Commit message: Resolve issue with robot's urdf.

File: vo_ros2_ws/src/robot_description/urdf/diffbot_camera.urdf.xacro (robot description, xacro)
@@ -35,4 +35,5 @@
   <link name="base_link">
     <visual>
+      <origin xyz="0 0 ${base_height/2}" rpy="0 0 0"/>
       <geometry>
         <cylinder radius="${base_radius}" length="${base_height}"/>
@@ -41,4 +42,5 @@
     </visual>
     <collision>
+      <origin xyz="0 0 ${base_height/2}" rpy="0 0 0"/>
       <geometry>
         <cylinder radius="${base_radius}" length="${base_height}"/>
@@ -46,4 +48,5 @@
     </collision>
     <inertial>
+      <origin xyz="0 0 ${base_height/2}" rpy="0 0 0"/>
       <mass value="2.0"/>
       <inertia ixx="0.0166" ixy="0" ixz="0"
